File: esp32-module/esp32-module.kicad_pcb (KiCad board)
At the start: 2 copper layers, 11 parts, among them IC1 ESP32-S3-WROOM-1-N4, J1 HTSW-104-08-G-S-RA, J2 HTSW-104-08-G-S-RA, U1 CP2102N-Axx-xQFN28

Commit message: Further Implementation
Parts:
- removed J1, J2: HTSW-104-08-G-S-RA, SamacSys_Parts:HDRRA4W64P0X254_1X4_1016X254X309P
- added C4: C10uf, Capacitor_SMD:C_0603_1608Metric, F.Cu at (102.2, 51.2)
- added C5: C100nf, Capacitor_SMD:C_0603_1608Metric, F.Cu at (78.6, 60.8)
- added C6: MAL214097803E3, SamacSys_Parts:CAPAE850X1050N, F.Cu at (84.6, 42.5)
- added C7: MAL214097803E3, SamacSys_Parts:CAPAE850X1050N, F.Cu at (107.1, 65.5)
- added IC2: LM1117MPX-3.3_NOPB, SamacSys_Parts:SOT230P700X180-4N, F.Cu at (107.5, 52.5)
- added LED1: APTD3216SECK, SamacSys_Parts:APTD3216SECK, F.Cu at (109.1, 59.0)
- added R3: 68R, Resistor_SMD:R_1206_3216Metric, F.Cu at (103.1, 59.0)
- added REF**: TestPoint_Pad_D2.0mm, TestPoint:TestPoint_Pad_D2.0mm, F.Cu at (100.5, 43.5)
- added REF**: TestPoint_Pad_D2.0mm, TestPoint:TestPoint_Pad_D2.0mm, F.Cu at (104.0, 43.5)
- added REF**: TestPoint_Pad_D2.0mm, TestPoint:TestPoint_Pad_D2.0mm, F.Cu at (97.0, 43.5)
- added REF**: TestPoint_Pad_D2.0mm, TestPoint:TestPoint_Pad_D2.0mm, F.Cu at (107.5, 43.5)
- added REF**: TestPoint_Pad_D2.0mm, TestPoint:TestPoint_Pad_D2.0mm, F.Cu at (111.0, 43.5)
- added REF**: TestPoint_Pad_D2.0mm, TestPoint:TestPoint_Pad_D2.0mm, F.Cu at (93.5, 43.5)
- moved R2 82.2 mm to (78.4, 66.3), turned to -90 degrees
- moved S1 76.6 mm to (84.8, 53.0), turned to 90 degrees
- moved C2 74.5 mm to (76.4, 67.1), turned to 90 degrees
- moved S2 72.5 mm to (95.5, 53.0), turned to 90 degrees
- moved IC1 52.7 mm to (90.1, 68.6)
- moved R1 51.3 mm to (105.1, 78.5), turned to 180 degrees
- moved C1 48.9 mm to (102.1, 78.5), turned to 90 degrees
- moved U1 48.6 mm to (107.6, 73.5)
- moved C3 48.5 mm to (102.1, 74.0), turned to 90 degrees
Connections:
- IC1 pad 13: Net-(IC1-IO19) -> unconnected-(IC1-IO19-Pad13)
- IC1 pad 14: Net-(IC1-IO20) -> unconnected-(IC1-IO20-Pad14)
- IC1 pad 28: unconnected-(IC1-IO35-Pad28) -> GPIO_35
- IC1 pad 29: unconnected-(IC1-IO36-Pad29) -> GPIO_36
- IC1 pad 30: unconnected-(IC1-IO37-Pad30) -> GPIO_37
- IC1 pad 31: unconnected-(IC1-IO38-Pad31) -> GPIO_38
- IC1 pad 32: unconnected-(IC1-IO39-Pad32) -> GPIO_39
- IC1 pad 33: unconnected-(IC1-IO40-Pad33) -> GPIO_40
- IC1 pad 34: unconnected-(IC1-IO41-Pad34) -> GPIO_41
- IC1 pad 35: unconnected-(IC1-IO42-Pad35) -> GPIO_42
- IC1 pad 4: unconnected-(IC1-IO4-Pad4) -> GPIO_4
- IC1 pad 5: unconnected-(IC1-IO5-Pad5) -> GPIO_5
- U1 pad 4: Net-(U1-D+) -> unconnected-(U1-D+-Pad4)
- U1 pad 5: Net-(U1-D-) -> unconnected-(U1-D--Pad5)
Routing:
- net RESET: track 0.00 -> 107.9 mm, vias 0 -> 2
- net +5V: track 0.00 -> 77.9 mm, vias 0 -> 2
- net ESP_UART_RX: track 0.00 -> 60.3 mm, vias 0 -> 2
- net unconnected-(IC1-IO20-Pad14): track 0.00 -> 59.7 mm, vias 0 -> 4
- net unconnected-(IC1-IO19-Pad13): track 0.00 -> 59.7 mm, vias 0 -> 2
- net ESP_UART_TX: track 0.00 -> 55.4 mm, vias 0 -> 2
- net unconnected-(U1-D--Pad5): track 0.00 -> 51.7 mm, vias 0 -> 2
- net ESP_UART_RTS: track 0.00 -> 50.6 mm, vias 0 -> 2
- net unconnected-(U1-D+-Pad4): track 0.00 -> 47.8 mm, vias 0 -> 2
- net VDD: track 0.00 -> 35.6 mm, vias 0 -> 7
- net ESP_UART_CTS: track 0.00 -> 31.7 mm, vias 0 -> 2
- net GPIO_35: track 0.00 -> 29.3 mm, vias 0 -> 2
- net BOOT: track 0.00 -> 29.3 mm
- net GPIO_42: track 0.00 -> 28.5 mm, vias 0 -> 2
- net GPIO_36: track 0.00 -> 28.4 mm, vias 0 -> 2
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- added copper zone on B.Cu, net GND
- added copper zone on F.Cu, net GND
Other:
- board outline added: 42.5 x 47.5 mm
- board text added: "+5v"
- board text added: "Boot"
- board text added: "CP2102N"
- board text added: "D+"
- board text added: "D-"
- board text added: "ESP USB OTG"
- board text added: "GND"
- board text added: "IO35"
- board text added: "IO36"
- board text added: "IO37"
- board text added: "IO38"
- board text added: "IO39"
- board text added: "IO4"
- board text added: "IO40"
- board text added: "IO41"
- board text added: "IO42"
- board text added: "IO5"
- board text added: "JLCJLCJLCJLC"
- board text added: "Reset"
- board text added: "VDD"
