File: esp32-module/esp32-module.kicad_sch (KiCad schematic)
At the start: 11 parts, among them IC1 ESP32-S3-WROOM-1-N4, J1 HTSW-104-08-G-S-RA, J2 HTSW-104-08-G-S-RA, U1 CP2102N-Axx-xQFN28

Commit message: Further Implementation
Parts:
- removed J1, J2: HTSW-104-08-G-S-RA, SamacSys_Parts:HDRRA4W64P0X254_1X4_1016X254X309P, symbol SamacSys_Parts:HTSW-104-08-G-S-RA
- added C4: C10uf, Capacitor_SMD:C_0603_1608Metric, symbol Device:C
- added C5: C100nf, Capacitor_SMD:C_0603_1608Metric, symbol Device:C
- added C6, C7: MAL214097803E3, CAPAE850X1050N, symbol SamacSys_Parts:MAL214097803E3
- added IC2: LM1117MPX-3.3_NOPB, SOT230P700X180-4N, symbol SamacSys_Parts:LM1117MPX-3.3_NOPB
- added LED1: APTD3216SECK, SamacSys_Parts:APTD3216SECK, symbol SamacSys_Parts:APTD3216SECK
- added R3: 68R, Resistor_SMD:R_1206_3216Metric, symbol Device:R
Connections:
- net +3.3V: now also C4.2, C5.1, C6.1, IC2.2 (OUTPUT), LED1.2
- net +5V: now also C7.1
- net GND: now also C4.1, C5.2, C6.2, C7.2, IC2.1 (ADJ/GND), R3.1
- net GPIO_35: now reaches IC1.28 (IO35)
- net GPIO_36: now reaches IC1.29 (IO36)
- net GPIO_37: now reaches IC1.30 (IO37)
- net GPIO_38: now reaches IC1.31 (IO38)
- net GPIO_39: now reaches IC1.32 (IO39)
- net GPIO_40: now reaches IC1.33 (IO40)
- net GPIO_41: now reaches IC1.34 (IO41)
- net GPIO_42: now reaches IC1.35 (IO42)
- net GPIO_4: now reaches IC1.4 (IO4)
- net GPIO_5: now reaches IC1.5 (IO5)
- new net: LED1.1, R3.2
- new net VDD: IC2.3 (INPUT)
Other:
- moved on the sheet: C1, C2, IC1, R1, R2, S1, S2, U1
